Commit message: the kobuki pkg was adjusted to add the batbot version of it also the echo sonar sim using LIDAR was added ...plus The LIDAR was adjusted to give 360 degree view

File: kobuki_description/urdf/kobuki_batbot.urdf.xacro (robot description, xacro)
@@ -8,5 +8,5 @@
 <robot name="kobuki" xmlns:xacro="http://ros.org/wiki/xacro">
   <xacro:include filename="$(find kobuki_description)/urdf/common_properties.urdf.xacro"/>
-  <xacro:include filename="$(find kobuki_description)/urdf/kobuki_gazebo.urdf.xacro"/>
+  <xacro:include filename="$(find kobuki_description)/urdf/kobuki_batbot_gazebo.urdf.xacro"/>
   <!-- Kobuki -->
   <xacro:macro name="kobuki">
@@ -150,5 +150,5 @@
       </inertial>
     </link>
-    <!-- Kobuki's sensors -->
+        <!-- Kobuki's sensors -->
     <joint name="gyro_joint" type="fixed">
       <axis xyz="0 1 0"/>
@@ -210,7 +210,8 @@
     <!-- Kobuki Gazebo simulation details -->
     <kobuki_sim/>
+    <!-- Kobuki Gazebo simulation details
+    <kobuki_sim/> -->
   </xacro:macro>
-  <!-- Lidar sensor -->
-  <xacro:include filename="$(find kobuki_description)/urdf/sensors/lidar_sensor.urdf.xacro" />
+  <xacro:include filename="$(find kobuki_description)/urdf/sensors/lidar_sensor.urdf.xacro"/>
   <xacro:lidar_sensor
     name="sonar2"
@@ -220,10 +221,10 @@
     min_range="0.06"
     max_range="20.0"
-    field_of_view_horizontal="${270*M_PI/180}"
+    field_of_view_horizontal="${360*M_PI/180}"
     field_of_view_vertical="${1*M_PI/180}"
     ray_count_horizontal="40"
     ray_count_vertical="1"
-    sensor_mesh="lidar_lite_v2_withRay/meshes/lidar_lite_v2_withRay.dae">
-    <origin xyz="0 0.0 0.5" rpy="0 0 0"/>
+    sensor_mesh="(find kobuki_description/meshes/lidar_lite_v2_withRay.dae">
+    <origin xyz="0 0.0 0.18" rpy="0 0 0"/>
   </xacro:lidar_sensor>
 </robot>

File: kobuki_description/urdf/kobuki_batbot_gazebo.urdf.xacro (robot description, xacro)
@@ -46,5 +46,5 @@
 	    </sensor>
 	  </gazebo>
-	  <gazebo reference="cliff_sensor_left_link">
+	 <gazebo reference="cliff_sensor_left_link">
 	    <sensor type="ray" name="cliff_sensor_left">
 	      <always_on>true</always_on>
@@ -136,29 +136,6 @@
 	    </sensor>
 	  </gazebo>
-	  <gazebo reference="gyro_link">
-	   <sensor type="imu" name="imu">
-        <always_on>true</always_on>
-        <update_rate>50</update_rate>
-        <visualize>false</visualize>
-        <imu>
-          <noise>
-            <type>gaussian</type>
-	          <rate>
-	            <mean>0.0</mean>
-	            <stddev>${0.0014*0.0014}</stddev> <!-- 0.25 x 0.25 (deg/s) -->
-	            <bias_mean>0.0</bias_mean>
-	            <bias_stddev>0.0</bias_stddev>
-	          </rate>
-		        <accel> <!-- not used in the plugin and real robot, hence using tutorial values -->
-			        <mean>0.0</mean>
-			        <stddev>1.7e-2</stddev>
-			        <bias_mean>0.1</bias_mean>
-			        <bias_stddev>0.001</bias_stddev>
-		        </accel>
-          </noise>
-	      </imu>
-      </sensor>
-	  </gazebo>
-	  <!-- <gazebo>
+<!--
+	  <gazebo>
 	    <plugin name="kobuki_controller" filename="libgazebo_ros_kobuki.so">
 	      <publish_tf>1</publish_tf>
@@ -177,5 +154,5 @@
 	    </plugin>
 	  </gazebo> -->
-	   <gazebo>
+    <gazebo>
     <plugin name="differential_drive_controller" filename="libgazebo_ros_diff_drive.so">
       <legacyMode>false</legacyMode>
